File: truelog.brd (EAGLE design)
At the start: 57.1 x 47 mm, 34 parts, among them IC1 LMV324, J2 ISP, Q1 MMBT2222A, Q2 MMBT2222A, Q3 MMBT2222A, Q4 MMBT2222A, U1 ATTINY84

Commit message: PCB eye candy
Parts:
- added U$1, U$2: (no value), my:POT-SYMBOL
Other:
- board text added: "9-15V DC"

Commit message: Logo added
Parts:
- added LOGO1: LOGO-MANTIS, my:LOGO-MANTIS
Changed lines of the file:
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@@
 <element name="U$1" library="my" package="POT-SYMBOL" value="" x="14.605" y="34.29" rot="R90"/>
 <element name="U$2" library="my" package="POT-SYMBOL" value="" x="29.845" y="34.29" rot="R90"/>
+<element name="LOGO1" library="my" package="LOGO-MANTIS" value="LOGO-MANTIS" x="50.8" y="8.255"/>
 </elements>
 <signals>
