File: truelog.sch (EAGLE design)
At the start: 34 parts, among them IC1 LMV324, J2 ISP, Q1 MMBT2222A, Q2 MMBT2222A, Q3 MMBT2222A, Q4 MMBT2222A, U1 ATTINY84

Commit message: Logo added
Parts:
- added LOGO1: LOGO-MANTIS, my:LOGO-MANTIS
Changed lines of the file:
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@@
 <part name="X2" library="con-wago-500" deviceset="W237-136" device=""/>
 <part name="J2" library="SparkFun-Connectors" deviceset="M06" device="LOCK" value="ISP"/>
+<part name="LOGO1" library="my" deviceset="LOGO-MANTIS" device=""/>
 </parts>
 <sheets>
@@
 <instance part="X2" gate="-6" x="63.5" y="99.06"/>
 <instance part="J2" gate="G$1" x="180.34" y="129.54"/>
+<instance part="LOGO1" gate="G$1" x="165.1" y="7.62"/>
 </instances>
 <busses>
